File: Drone_LM5145.kicad_pcb (KiCad board)
At the start: 2 copper layers, 45 x 22 mm, 53 parts, among them Q1 BSC070N10, Q2 BSC070N10, U1 LM5145, U2 LMR51610

Commit message: 更新ibom和加工文件
Parts:
- C17: value C_Polarized -> 100uF 63V
- C18, C20: value 220u -> 220uF 35V
- C19: value 220u -> 100uF 63V
- C21: value C_Small -> 100n
Changed lines of the file:
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@@
 			)
 		)
-		(property "Value" "C_Small"
+		(property "Value" "100n"
 			(at 0 1.43 90)
 			(layer "F.Fab")
@@
 			)
 		)
-		(property "Value" "220u"
+		(property "Value" "220uF 35V"
 			(at 1.75 -5.25 90)
 			(layer "B.Fab")
@@
 			)
 		)
-		(property "Value" "220u"
+		(property "Value" "220uF 35V"
 			(at 1.75 -5.25 90)
 			(layer "B.Fab")
@@
 			)
 		)
-		(property "Value" "C_Polarized"
+		(property "Value" "100uF 63V"
 			(at 1.75 -5.25 -90)
 			(layer "B.Fab")
@@
 			)
 		)
-		(property "Value" "220u"
+		(property "Value" "100uF 63V"
 			(at 1.75 -5.25 -90)
 			(layer "B.Fab")
