File: Drone_LM5145.kicad_sch (KiCad schematic)
At the start: 53 parts, among them Q1 BSC070N10, Q2 BSC070N10, U1 LM5145, U2 LMR51610

Commit message: 更新ibom和加工文件
Parts:
- C21: value C_Small -> 100n
Changed lines of the file:
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@@
 			)
 		)
-		(property "Value" "C_Small"
+		(property "Value" "100n"
 			(at 168.91 54.6035 0)
 			(effects
